File: keeb60.kicad_pcb (KiCad board)
At the start: 2 copper layers, 124 parts, among them J1 Battery Connector, K000 Esc, K001 1, K002 2, K003 3, K004 4, K005 5, K006 6, K007 7, K008 8, K009 9, K010 0, K011 _, K012 =, K013 Backspace, K100 Tab, K101 Q, K102 W, K103 E, K104 R, K105 T, K106 Y, K107 U, K108 I, K109 O, K110 P, K111 [, K112 ], K113 |, K200 Caps Lock, K201 A, K202 S, K203 D, K204 F, K205 G, K206 H, K207 J, K208 K, K209 L, K210 ;, K211 ,, K213 Enter, K300 Shift, K302 Z, K303 X, K304 C, K305 V, K306 B, K307 N, K308 M, K309 ,, K310 ., K311 /, K313 Shift, K400 Ctrl, K401 Option, K402 Command, K406 Space, K410 Command, K411 Option, K412 Function, K413 Ctrl, U1 ProMicro

Commit message: Start placing diodes
Parts:
- D0, D1, D10, D11, D12, D13, D14, D15, D16, D17, D18, D19, D2, D20, D21, D22, D23, D24, D25, D26, D27, D28, D29, D3, D30, D31, D32, D33, D34, D35, D36, D37, D38, D39, D4, D40, D41, D42, D43, D44, D45, D46, D47, D48, D49, D5, D50, D51, D52, D53, D54, D55, D56, D57, D58, D59, D6, D60, D7, D8, D9, J1: moved to F.Cu
- U1: moved to B.Cu
- moved J1 293.5 mm to (224.2, 267.0), turned to 0 degrees
- moved U1 276.2 mm to (192.4, 262.6), turned to 180 degrees
- moved K113 261.8 mm to (329.9, 163.5)
- moved K012 258.4 mm to (296.5, 144.5)
- moved K011 248.8 mm to (277.5, 144.5)
- moved K112 246.2 mm to (306.1, 163.5)
- moved K010 240.8 mm to (258.4, 144.5)
- moved K111 236.3 mm to (287.0, 163.5)
- moved K213 234.9 mm to (322.7, 182.6)
- moved K110 228.0 mm to (268.0, 163.5)
- moved K013 222.8 mm to (325.1, 144.5)
- moved K109 221.4 mm to (248.9, 163.5)
- moved K303 220.4 mm to (129.9, 201.6)
- moved K108 216.8 mm to (229.9, 163.5)
- moved K107 214.3 mm to (210.8, 163.5)
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
Commit message: All diodes positioned
Parts:
- moved D60 210.1 mm to (338.1, 225.4), turned to 90 degrees
- moved D27 198.0 mm to (336.6, 168.2), turned to 90 degrees
- moved D59 196.9 mm to (314.3, 225.4), turned to 90 degrees
- moved D54 194.3 mm to (100.0, 225.5), turned to 90 degrees
- moved D40 190.4 mm to (328.6, 187.3), turned to 90 degrees
- moved D52 188.4 mm to (323.9, 206.4), turned to 90 degrees
- moved D13 186.7 mm to (331.0, 149.2), turned to 90 degrees
- moved D58 185.9 mm to (290.5, 225.4), turned to 90 degrees
- moved D55 181.0 mm to (123.8, 225.4), turned to 90 degrees
- moved D53 178.7 mm to (76.3, 225.4), turned to 90 degrees
- moved D57 177.5 mm to (266.7, 225.4), turned to 90 degrees
- moved D39 169.8 mm to (297.7, 187.3), turned to 90 degrees
- moved D26 167.5 mm to (311.9, 168.2), turned to 90 degrees
- moved D51 166.7 mm to (288.1, 206.4), turned to 90 degrees
- moved D41 165.1 mm to (85.7, 206.4), turned to 90 degrees
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
Commit message: Move diodes to correct layers
Parts:
- D0, D1, D10, D11, D12, D13, D2, D27, D28, D3, D30, D31, D32, D33, D34, D35, D36, D37, D38, D39, D4, D40, D41, D42, D43, D44, D45, D46, D47, D48, D49, D5, D50, D51, D52, D53, D54, D55, D56, D57, D58, D59, D6, D60, D7, D8, D9, J1: moved to B.Cu
- U1: moved to F.Cu
- turned J1 to 180 degrees
- turned U1 to 0 degrees

Commit message: Changes
Parts:
- moved J1 81.0 mm to (158.8, 219.2), turned to -90 degrees
- moved U1 46.8 mm to (216.9, 219.5), turned to 90 degrees

Commit message: Remove JST from board
Parts:
- removed J1: Battery Connector, Connector_JST:JST_XH_B2B-XH-A_1x02_P2.50mm_Vertical
- moved D53 53.1 mm to (92.7, 174.9)
- moved D54 53.1 mm to (116.5, 175.0)
- moved D55 53.1 mm to (140.3, 174.9)
- moved D56 53.1 mm to (211.7, 174.9)
- moved D57 53.1 mm to (283.2, 174.9)
- moved D58 53.1 mm to (307.0, 174.9)
- moved D59 53.1 mm to (330.8, 174.9)
- moved D60 53.1 mm to (354.6, 174.9)
- moved K300 53.1 mm to (96.3, 151.1)
- moved K302 53.1 mm to (127.3, 151.1)
- moved K303 53.1 mm to (146.3, 151.1)
- moved K304 53.1 mm to (165.4, 151.1)
- moved K305 53.1 mm to (184.4, 151.1)
- moved K306 53.1 mm to (203.5, 151.1)
- moved K307 53.1 mm to (222.5, 151.1)
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
Commit message: Move to 13 columns
Parts:
- D0, D1, D10, D11, D12, D13, D2, D27, D28, D3, D30, D31, D32, D33, D34, D35, D36, D37, D38, D39, D4, D40, D41, D42, D43, D44, D45, D46, D47, D48, D49, D5, D50, D51, D52, D53, D54, D55, D56, D57, D58, D59, D6, D60, D7, D8, D9: moved to F.Cu
- K113: value | -> Pipe
- moved K113 205.5 mm to (144.9, 153.2)
- moved K012 185.9 mm to (128.1, 113.0)
- moved K112 180.2 mm to (144.9, 143.2)
- moved K009 170.0 mm to (111.3, 183.4)
- moved K011 166.1 mm to (128.1, 102.9)
- moved K111 159.9 mm to (144.9, 133.1)
- moved D13 156.9 mm to (212.9, 179.4), turned to 0 degrees
- moved K413 155.9 mm to (195.2, 143.2)
- moved K211 152.3 mm to (161.7, 173.3)
- moved K008 148.5 mm to (111.3, 173.3)
- moved K010 146.8 mm to (128.1, 92.9)
- moved D53 144.5 mm to (236.1, 192.8), turned to 0 degrees
- moved K110 139.9 mm to (144.9, 123.1)
- moved D27 137.3 mm to (224.5, 166.0), turned to 0 degrees
- moved K412 134.9 mm to (195.2, 133.1)
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Connections:
- D0 pad 1: /Row0 -> Row0
- D1 pad 1: /Row0 -> Row0
- D10 pad 1: /Row0 -> Row0
- D11 pad 1: /Row0 -> Row0
- D12 pad 1: /Row0 -> Row0
- D13 pad 1: /Row0 -> Row1
- D14 pad 1: /Row1 -> Row1
- D15 pad 1: /Row1 -> Row1
- D16 pad 1: /Row1 -> Row1
- D17 pad 1: /Row1 -> Row1
- D18 pad 1: /Row1 -> Row1
- D19 pad 1: /Row1 -> Row1
- D2 pad 1: /Row0 -> Row0
- D20 pad 1: /Row1 -> Row1
- D21 pad 1: /Row1 -> Row1
- D22 pad 1: /Row1 -> Row1
- D23 pad 1: /Row1 -> Row1
- D24 pad 1: /Row1 -> Row1
- D25 pad 1: /Row1 -> Row1
- D26 pad 1: /Row1 -> Row2
- D27 pad 1: /Row1 -> Row2
- D28 pad 1: /Row2 -> Row2
- D29 pad 1: /Row2 -> Row2
- D3 pad 1: /Row0 -> Row0
- D30 pad 1: /Row2 -> Row2
- D31 pad 1: /Row2 -> Row2
- D32 pad 1: /Row2 -> Row2
- D33 pad 1: /Row2 -> Row2
- D34 pad 1: /Row2 -> Row2
- D35 pad 1: /Row2 -> Row2
- D36 pad 1: /Row2 -> Row2
- D37 pad 1: /Row2 -> Row2
- D38 pad 1: /Row2 -> Row2
- D39 pad 1: /Row2 -> Row3
- D4 pad 1: /Row0 -> Row0
- D40 pad 1: /Row2 -> Row3
- D41 pad 1: /Row3 -> Row3
- D42 pad 1: /Row3 -> Row3
- D43 pad 1: /Row3 -> Row3
- D44 pad 1: /Row3 -> Row3
- D45 pad 1: /Row3 -> Row3
- D46 pad 1: /Row3 -> Row3
- D47 pad 1: /Row3 -> Row3
- D48 pad 1: /Row3 -> Row3
- D49 pad 1: /Row3 -> Row3
- D5 pad 1: /Row0 -> Row0
- D50 pad 1: /Row3 -> Row3
- D51 pad 1: /Row3 -> /Row4
- D52 pad 1: /Row3 -> /Row4
- D6 pad 1: /Row0 -> Row0
- D7 pad 1: /Row0 -> Row0
- D8 pad 1: /Row0 -> Row0
- D9 pad 1: /Row0 -> Row0
- K013 pad 1: Net-(D13-A) -> Net-(D56-A)
- K013 pad 2: /Col13 -> /Col8
- K100 pad 1: Net-(D14-A) -> Net-(D13-A)
- K101 pad 1: Net-(D15-A) -> Net-(D14-A)
- K102 pad 1: Net-(D16-A) -> Net-(D15-A)
- K103 pad 1: Net-(D17-A) -> Net-(D16-A)
- K104 pad 1: Net-(D18-A) -> Net-(D17-A)
- K105 pad 1: Net-(D19-A) -> Net-(D18-A)
- K106 pad 1: Net-(D20-A) -> Net-(D19-A)
- K107 pad 1: Net-(D21-A) -> Net-(D20-A)
- K108 pad 1: Net-(D22-A) -> Net-(D21-A)
- K109 pad 1: Net-(D23-A) -> Net-(D22-A)
- K110 pad 1: Net-(D24-A) -> Net-(D23-A)
- K111 pad 1: Net-(D25-A) -> Net-(D24-A)
- K112 pad 1: Net-(D26-A) -> Net-(D25-A)
- K113 pad 1: Net-(D27-A) -> Net-(D55-A)
- K113 pad 2: /Col13 -> /Col7
- K200 pad 1: Net-(D28-A) -> Net-(D26-A)
- K201 pad 1: Net-(D29-A) -> Net-(D27-A)
- K202 pad 1: Net-(D30-A) -> Net-(D28-A)
- K203 pad 1: Net-(D31-A) -> Net-(D29-A)
- K204 pad 1: Net-(D32-A) -> Net-(D30-A)
- K205 pad 1: Net-(D33-A) -> Net-(D31-A)
- K206 pad 1: Net-(D34-A) -> Net-(D32-A)
- K207 pad 1: Net-(D35-A) -> Net-(D33-A)
- K208 pad 1: Net-(D36-A) -> Net-(D34-A)
- K209 pad 1: Net-(D37-A) -> Net-(D35-A)
- K210 pad 1: Net-(D38-A) -> Net-(D36-A)
- K211 pad 1: Net-(D39-A) -> Net-(D37-A)
- K213 pad 1: Net-(D40-A) -> Net-(D38-A)
- K213 pad 2: /Col13 -> /Col12
- K300 pad 1: Net-(D41-A) -> Net-(D39-A)
- K302 pad 1: Net-(D42-A) -> Net-(D40-A)
- K303 pad 1: Net-(D43-A) -> Net-(D41-A)
- K304 pad 1: Net-(D44-A) -> Net-(D42-A)
- K305 pad 1: Net-(D45-A) -> Net-(D43-A)
- K306 pad 1: Net-(D46-A) -> Net-(D44-A)
- K307 pad 1: Net-(D47-A) -> Net-(D45-A)
- K308 pad 1: Net-(D48-A) -> Net-(D46-A)
- K309 pad 1: Net-(D49-A) -> Net-(D47-A)
- K310 pad 1: Net-(D50-A) -> Net-(D48-A)
- K311 pad 1: Net-(D51-A) -> Net-(D49-A)
- K313 pad 1: Net-(D52-A) -> Net-(D50-A)
- K313 pad 2: /Col13 -> /Col12
- K400 pad 1: Net-(D53-A) -> Net-(D51-A)
- K401 pad 1: Net-(D54-A) -> Net-(D52-A)
- K402 pad 1: Net-(D55-A) -> Net-(D53-A)
- K406 pad 1: Net-(D56-A) -> Net-(D54-A)
- K410 pad 2: /Col10 -> /Col9
- K411 pad 2: /Col11 -> /Col10
- K412 pad 2: /Col12 -> /Col11
- K413 pad 2: /Col13 -> /Col12
- U1 pad 1: /Col0 -> unconnected-(U1-GP0(TX)-Pad1)
- U1 pad 10: /Row0 -> unconnected-(U1-GP7-Pad10)
- U1 pad 11: /Row1 -> unconnected-(U1-GP8-Pad11)
- U1 pad 12: /Row2 -> unconnected-(U1-GP9-Pad12)
- U1 pad 13: /Row3 -> unconnected-(U1-GP21-Pad13)
- U1 pad 14: /Col7 -> unconnected-(U1-GP23-Pad14)
- U1 pad 15: /Col8 -> unconnected-(U1-GP20-Pad15)
- U1 pad 16: /Col9 -> unconnected-(U1-GP22-Pad16)
- U1 pad 17: /Col10 -> unconnected-(U1-GP26(A0)-Pad17)
- U1 pad 18: /Col11 -> unconnected-(U1-GP27(A1)-Pad18)
- U1 pad 19: /Col12 -> unconnected-(U1-GP28(A2)-Pad19)
- U1 pad 2: /Col1 -> unconnected-(U1-GP1(RX)-Pad2)
- U1 pad 20: /Col13 -> unconnected-(U1-GP29(A3)-Pad20)
- U1 pad 23: Net-(J1-Pin_1) -> unconnected-(U1-GND-Pad23)
- U1 pad 3: unconnected-(U1-GND-Pad3) -> GND
- U1 pad 4: unconnected-(U1-GND-Pad4) -> GND
- U1 pad 5: /Col2 -> Row2
- U1 pad 6: /Col3 -> unconnected-(U1-SCL(GP3)-Pad6)
- U1 pad 7: /Col4 -> unconnected-(U1-GP4-Pad7)
- U1 pad 8: /Col5 -> unconnected-(U1-GP5-Pad8)
- U1 pad 9: /Col6 -> unconnected-(U1-GP6-Pad9)

Commit message: Fix alignment, bah!
Parts:
- D0, D1, D2, D3, D4: moved to B.Cu
- moved D0 256.7 mm to (-40.5, 98.4), turned to 90 degrees
- moved K300 253.4 mm to (-34.1, 150.8)
- moved D1 239.3 mm to (-21.4, 98.4), turned to 90 degrees
- moved K401 228.4 mm to (-19.8, 169.9)
- moved K400 222.5 mm to (-43.7, 169.9)
- moved D2 222.3 mm to (-2.38, 98.4), turned to 90 degrees
- moved D3 205.7 mm to (16.7, 98.4), turned to 90 degrees
- moved K402 202.6 mm to (3.97, 169.9)
- moved D4 189.6 mm to (35.7, 98.4), turned to 90 degrees
- moved K200 186.5 mm to (-38.9, 131.8)
- moved K303 172.6 mm to (15.9, 150.8)
- moved K100 169.7 mm to (-41.3, 112.7)
- moved K302 168.0 mm to (-3.17, 150.8)
- moved U1 165.4 mm to (104.8, 168.6), turned to 90 degrees
- moved K201 163.0 mm to (-12.7, 131.8)
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Connections:
- D0 pad 1: Row0 -> (no net)
- D0 pad 2: Net-(D0-A) -> (no net)
- D1 pad 1: Row0 -> (no net)
- D1 pad 2: Net-(D1-A) -> (no net)
- D2 pad 1: Row0 -> (no net)
- D2 pad 2: Net-(D2-A) -> (no net)
- D3 pad 1: Row0 -> (no net)
- D3 pad 2: Net-(D3-A) -> (no net)
- D4 pad 1: Row0 -> (no net)
- D4 pad 2: Net-(D4-A) -> (no net)
- D51 pad 1: /Row4 -> Row4
- D52 pad 1: /Row4 -> Row4
- D53 pad 1: /Row4 -> Row4
- D54 pad 1: /Row4 -> Row4
- D55 pad 1: /Row4 -> Row4
- D56 pad 1: /Row4 -> Row4
- D57 pad 1: /Row4 -> Row4
- D58 pad 1: /Row4 -> Row4
- D59 pad 1: /Row4 -> Row4
- D60 pad 1: /Row4 -> Row4
- K000 pad 2: /Col0 -> Col0
- K001 pad 2: /Col1 -> Col1
- K002 pad 2: /Col2 -> Col2
- K003 pad 2: /Col3 -> Col3
- K004 pad 2: /Col4 -> Col4
- K005 pad 2: /Col5 -> Col5
- K006 pad 2: /Col6 -> Col6
- K007 pad 2: /Col7 -> Col7
- K008 pad 2: /Col8 -> Col8
- K009 pad 2: /Col9 -> Col9
- K010 pad 2: /Col10 -> Col10
- K011 pad 2: /Col11 -> Col11
- K012 pad 2: /Col12 -> Col12
- K013 pad 1: Net-(D56-A) -> Net-(D60-A)
- K013 pad 2: /Col8 -> Col12
- K100 pad 2: /Col0 -> Col0
- K101 pad 1: Net-(D14-A) -> (no net)
- K101 pad 2: /Col1 -> (no net)
- K102 pad 2: /Col2 -> Col2
- K103 pad 2: /Col3 -> Col3
- K104 pad 2: /Col4 -> Col4
- K105 pad 2: /Col5 -> Col5
- K106 pad 2: /Col6 -> Col6
- K107 pad 2: /Col7 -> Col7
- K108 pad 2: /Col8 -> Col8
- K109 pad 2: /Col9 -> Col9
- K110 pad 2: /Col10 -> Col10
- K111 pad 2: /Col11 -> Col11
- K112 pad 2: /Col12 -> Col12
- K113 pad 1: Net-(D55-A) -> Net-(D59-A)
- K113 pad 2: /Col7 -> Col11
- K200 pad 2: /Col0 -> Col0
- K201 pad 2: /Col1 -> Col1
- K202 pad 2: /Col2 -> Col2
- K203 pad 2: /Col3 -> Col3
- K204 pad 1: Net-(D30-A) -> (no net)
- K204 pad 2: /Col4 -> (no net)
- K205 pad 2: /Col5 -> Col5
- K206 pad 2: /Col6 -> Col6
- K207 pad 2: /Col7 -> Col7
- K208 pad 2: /Col8 -> Col8
- K209 pad 1: Net-(D35-A) -> (no net)
- K209 pad 2: /Col9 -> (no net)
- K210 pad 2: /Col10 -> Col10
- K211 pad 2: /Col11 -> Col11
- K213 pad 2: /Col12 -> Col12
- K300 pad 2: /Col0 -> Col0
- K302 pad 2: /Col2 -> Col2
- K303 pad 2: /Col3 -> Col3
- K304 pad 2: /Col4 -> Col4
- K305 pad 2: /Col5 -> Col5
- K306 pad 2: /Col6 -> Col6
- K307 pad 2: /Col7 -> Col7
- K308 pad 2: /Col8 -> Col8
- K309 pad 2: /Col9 -> Col9
- K310 pad 2: /Col10 -> Col10
- K311 pad 2: /Col11 -> Col11
- K313 pad 2: /Col12 -> Col12
- K400 pad 2: /Col0 -> Col0
- K401 pad 2: /Col1 -> Col1
- K402 pad 2: /Col2 -> Col2
- K406 pad 2: /Col6 -> Col6
- K410 pad 1: Net-(D57-A) -> Net-(D55-A)
- K410 pad 2: /Col9 -> Col7
- K411 pad 1: Net-(D58-A) -> Net-(D56-A)
- K411 pad 2: /Col10 -> Col8
- K412 pad 1: Net-(D59-A) -> Net-(D57-A)
- K412 pad 2: /Col11 -> Col9
- K413 pad 1: Net-(D60-A) -> Net-(D58-A)
- K413 pad 2: /Col12 -> Col10
- U1 pad 1: unconnected-(U1-GP0(TX)-Pad1) -> Row0
- U1 pad 10: unconnected-(U1-GP7-Pad10) -> Col2
- U1 pad 11: unconnected-(U1-GP8-Pad11) -> Col3
- U1 pad 12: unconnected-(U1-GP9-Pad12) -> Col4
- U1 pad 13: unconnected-(U1-GP21-Pad13) -> Col12
- U1 pad 14: unconnected-(U1-GP23-Pad14) -> Col11
- U1 pad 15: unconnected-(U1-GP20-Pad15) -> Col10
- U1 pad 16: unconnected-(U1-GP22-Pad16) -> Col9
- U1 pad 17: unconnected-(U1-GP26(A0)-Pad17) -> Col8
- U1 pad 18: unconnected-(U1-GP27(A1)-Pad18) -> Col7
- U1 pad 19: unconnected-(U1-GP28(A2)-Pad19) -> Col6
- U1 pad 2: unconnected-(U1-GP1(RX)-Pad2) -> Row1
- U1 pad 20: unconnected-(U1-GP29(A3)-Pad20) -> Col5
- U1 pad 24: unconnected-(U1-5V-Pad24) -> Net-(U1-5V)
- U1 pad 6: unconnected-(U1-SCL(GP3)-Pad6) -> Row3
- U1 pad 7: unconnected-(U1-GP4-Pad7) -> Row4
- U1 pad 8: unconnected-(U1-GP5-Pad8) -> Col0
- U1 pad 9: unconnected-(U1-GP6-Pad9) -> Col1

Commit message: Position diodes
Parts:
- D10, D11, D12, D13, D14, D15, D16, D17, D18, D19, D20, D21, D22, D23, D24, D25, D26, D27, D28, D29, D30, D31, D32, D33, D34, D35, D36, D37, D38, D39, D40, D41, D42, D43, D44, D45, D46, D47, D48, D49, D5, D50, D51, D52, D53, D54, D55, D56, D57, D58, D59, D6, D60, D7, D8, D9: moved to B.Cu
- moved D53 211.4 mm to (69.1, 177.0), turned to 90 degrees
- moved D54 197.4 mm to (92.9, 177.0), turned to 90 degrees
- moved D41 195.6 mm to (78.6, 158.0), turned to 90 degrees
- moved D28 194.4 mm to (73.8, 138.9), turned to 90 degrees
- moved D14 187.8 mm to (71.4, 119.9), turned to 90 degrees
- moved D55 173.5 mm to (116.7, 177.0), turned to 90 degrees
- moved D29 168.2 mm to (100.0, 138.9), turned to 90 degrees
- moved D15 165.0 mm to (95.2, 119.9), turned to 90 degrees
- moved D42 164.5 mm to (109.5, 158.0), turned to 90 degrees
- moved D30 149.3 mm to (119.1, 138.9), turned to 90 degrees
- moved D16 147.3 mm to (114.3, 119.9), turned to -90 degrees
- moved D43 145.4 mm to (128.6, 158.0), turned to -90 degrees
- moved D31 130.4 mm to (138.1, 138.9), turned to 90 degrees
- moved D17 130.0 mm to (133.3, 119.9), turned to 90 degrees
- moved D44 126.4 mm to (147.6, 158.0), turned to 90 degrees
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Connections:
- D10 pad 1: Row0 -> (no net)
- D10 pad 2: Net-(D10-A) -> (no net)
- D11 pad 1: Row0 -> (no net)
- D11 pad 2: Net-(D11-A) -> (no net)
- D12 pad 1: Row0 -> (no net)
- D12 pad 2: Net-(D12-A) -> (no net)
- D13 pad 1: Row1 -> (no net)
- D13 pad 2: Net-(D13-A) -> (no net)
- D14 pad 1: Row1 -> (no net)
- D14 pad 2: Net-(D14-A) -> (no net)
- D15 pad 1: Row1 -> (no net)
- D15 pad 2: Net-(D15-A) -> (no net)
- D16 pad 1: Row1 -> (no net)
- D16 pad 2: Net-(D16-A) -> (no net)
- D17 pad 1: Row1 -> (no net)
- D17 pad 2: Net-(D17-A) -> (no net)
- D18 pad 1: Row1 -> (no net)
- D18 pad 2: Net-(D18-A) -> (no net)
- D19 pad 1: Row1 -> (no net)
- D19 pad 2: Net-(D19-A) -> (no net)
- D20 pad 1: Row1 -> (no net)
- D20 pad 2: Net-(D20-A) -> (no net)
- D21 pad 1: Row1 -> (no net)
- D21 pad 2: Net-(D21-A) -> (no net)
- D22 pad 1: Row1 -> (no net)
- D22 pad 2: Net-(D22-A) -> (no net)
- D23 pad 1: Row1 -> (no net)
- D23 pad 2: Net-(D23-A) -> (no net)
- D24 pad 1: Row1 -> (no net)
- D24 pad 2: Net-(D24-A) -> (no net)
- D25 pad 1: Row1 -> (no net)
- D25 pad 2: Net-(D25-A) -> (no net)
- D26 pad 1: Row2 -> (no net)
- D26 pad 2: Net-(D26-A) -> (no net)
- D27 pad 1: Row2 -> (no net)
- D27 pad 2: Net-(D27-A) -> (no net)
- D28 pad 1: Row2 -> (no net)
- D28 pad 2: Net-(D28-A) -> (no net)
- D29 pad 1: Row2 -> (no net)
- D29 pad 2: Net-(D29-A) -> (no net)
- D30 pad 1: Row2 -> (no net)
- D30 pad 2: Net-(D30-A) -> (no net)
- D31 pad 1: Row2 -> (no net)
- D31 pad 2: Net-(D31-A) -> (no net)
- D32 pad 1: Row2 -> (no net)
- D32 pad 2: Net-(D32-A) -> (no net)
- D33 pad 1: Row2 -> (no net)
- D33 pad 2: Net-(D33-A) -> (no net)
- D34 pad 1: Row2 -> (no net)
- D34 pad 2: Net-(D34-A) -> (no net)
- D35 pad 1: Row2 -> (no net)
- D35 pad 2: Net-(D35-A) -> (no net)
- D36 pad 1: Row2 -> (no net)
- D36 pad 2: Net-(D36-A) -> (no net)
- D37 pad 1: Row2 -> (no net)
- D37 pad 2: Net-(D37-A) -> (no net)
- D38 pad 1: Row2 -> (no net)
- D38 pad 2: Net-(D38-A) -> (no net)
- D39 pad 1: Row3 -> (no net)
- D39 pad 2: Net-(D39-A) -> (no net)
- D40 pad 1: Row3 -> (no net)
- D40 pad 2: Net-(D40-A) -> (no net)
- D41 pad 1: Row3 -> (no net)
- D41 pad 2: Net-(D41-A) -> (no net)
- D42 pad 1: Row3 -> (no net)
- D42 pad 2: Net-(D42-A) -> (no net)
- D43 pad 1: Row3 -> (no net)
- D43 pad 2: Net-(D43-A) -> (no net)
- D44 pad 1: Row3 -> (no net)
- D44 pad 2: Net-(D44-A) -> (no net)
- D45 pad 1: Row3 -> (no net)
- D45 pad 2: Net-(D45-A) -> (no net)
- D46 pad 1: Row3 -> (no net)
- D46 pad 2: Net-(D46-A) -> (no net)
- D47 pad 1: Row3 -> (no net)
- D47 pad 2: Net-(D47-A) -> (no net)
- D48 pad 1: Row3 -> (no net)
- D48 pad 2: Net-(D48-A) -> (no net)
- D49 pad 1: Row3 -> (no net)
- D49 pad 2: Net-(D49-A) -> (no net)
- D5 pad 1: Row0 -> (no net)
- D5 pad 2: Net-(D5-A) -> (no net)
- D50 pad 1: Row3 -> (no net)
- D50 pad 2: Net-(D50-A) -> (no net)
- D51 pad 1: Row4 -> (no net)
- D51 pad 2: Net-(D51-A) -> (no net)
- D52 pad 1: Row4 -> (no net)
- D52 pad 2: Net-(D52-A) -> (no net)
- D53 pad 1: Row4 -> (no net)
- D53 pad 2: Net-(D53-A) -> (no net)
- D54 pad 1: Row4 -> (no net)
- D54 pad 2: Net-(D54-A) -> (no net)
- D55 pad 1: Row4 -> (no net)
- D55 pad 2: Net-(D55-A) -> (no net)
- D56 pad 1: Row4 -> (no net)
- D56 pad 2: Net-(D56-A) -> (no net)
- D57 pad 1: Row4 -> (no net)
- D57 pad 2: Net-(D57-A) -> (no net)
- D58 pad 1: Row4 -> (no net)
- D58 pad 2: Net-(D58-A) -> (no net)
- D59 pad 1: Row4 -> (no net)
- D59 pad 2: Net-(D59-A) -> (no net)
- D6 pad 1: Row0 -> (no net)
- D6 pad 2: Net-(D6-A) -> (no net)
- D60 pad 1: Row4 -> (no net)
- D60 pad 2: Net-(D60-A) -> (no net)
- D7 pad 1: Row0 -> (no net)
- D7 pad 2: Net-(D7-A) -> (no net)
- D8 pad 1: Row0 -> (no net)
- D8 pad 2: Net-(D8-A) -> (no net)
- D9 pad 1: Row0 -> (no net)
- D9 pad 2: Net-(D9-A) -> (no net)
