File: keeb60.kicad_pcb (KiCad board)
At the start: 2 copper layers, 290 x 99.2 mm, 127 parts, among them K000 Esc, K001 1, K002 2, K003 3, K004 4, K005 5, K006 6, K007 7, K008 8, K009 9, K010 0, K011 _, K012 =, K013 Backspace, K100 Tab, K101 Q, K102 W, K103 E, K104 R, K105 T, K106 Y, K107 U, K108 I, K109 O, K110 P, K111 [, K112 ], K113 Pipe, K200 Caps Lock, K201 A, K202 S, K203 D, K204 F, K205 G, K206 H, K207 J, K208 K, K209 L, K210 ;, K211 ,, K213 Enter, K300 Shift, K302 Z, K303 X, K304 C, K305 V, K306 B, K307 N, K308 M, K309 ,, K310 ., K311 /, K313 Shift, K400 Ctrl, K401 Option, K402 Command, K406 Space, K410 Command, K411 Option, K412 Function, K413 Ctrl, U1 ProMicro

Commit message: Fix DRC. V1.3
Routing:
- net Row4: track 383.5 -> 382.8 mm
Changed lines of the file:
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@@
 	)
 	(segment
-		(start 62.48375 140.55625)
-		(end 62.70625 140.55625)
-		(width 0.254)
-		(layer "B.Cu")
-		(net 32)
-	)
-	(segment
 		(start 222.46 179.86375)
 		(end 219.9845 177.38825)
@@
 	)
 	(segment
-		(start 234.750223 168.041732)
-		(end 233.595769 168.041731)
+		(start 218.257981 168.041731)
+		(end 234.750223 168.041732)
 		(width 0.254)
 		(layer "F.Cu")
@@
 		(net 73)
 	)
-	(segment
-		(start 233.595769 168.041731)
-		(end 218.257981 168.041731)
-		(width 0.254)
-		(layer "F.Cu")
-		(net 73)
-	)
 	(via
 		(at 200.31075 90.96375)
@@
 	)
 	(segment
-		(start 330.93125 178.65625)
-		(end 334.16875 175.41875)
+		(start 57.94375 178.65625)
+		(end 105.56875 178.65625)
 		(width 0.254)
 		(layer "B.Cu")
@@
 	)
 	(segment
-		(start 57.94375 178.65625)
-		(end 105.56875 178.65625)
+		(start 331.725 121.50625)
+		(end 334.16875 123.95)
 		(width 0.254)
 		(layer "B.Cu")
@@
 	)
 	(segment
-		(start 327.98 121.50625)
-		(end 317.5 121.50625)
+		(start 317.5 121.50625)
+		(end 331.725 121.50625)
 		(width 0.254)
 		(layer "B.Cu")
@@
 	)
 	(segment
-		(start 107.21875 177.00625)
-		(end 175.35625 177.00625)
+		(start 334.16875 123.95)
+		(end 334.16875 175.41875)
 		(width 0.254)
 		(layer "B.Cu")
@@
 	)
 	(segment
-		(start 328.68375 121.50625)
-		(end 327.98 121.50625)
-		(width 0.2)
-		(layer "B.Cu")
-		(net 82)
-	)
-	(segment
-		(start 319.88125 178.65625)
-		(end 330.93125 178.65625)
+		(start 107.21875 177.00625)
+		(end 175.35625 177.00625)
 		(width 0.254)
 		(layer "B.Cu")
@@
 	(segment
 		(start 334.16875 175.41875)
-		(end 334.16875 123.95)
+		(end 330.93125 178.65625)
 		(width 0.254)
 		(layer "B.Cu")
@@
 	)
 	(segment
+		(start 330.93125 178.65625)
+		(end 319.88125 178.65625)
+		(width 0.254)
+		(layer "B.Cu")
+		(net 82)
+	)
+	(segment
 		(start 306.99 113.93)
 		(end 312.7375 108.1825)
@@
 		(width 0.254)
 		(layer "B.Cu")
-		(net 82)
-	)
-	(segment
-		(start 331.725 121.50625)
-		(end 334.16875 123.95)
-		(width 0.254)
-		(layer "B.Cu")
-		(net 82)
-	)
-	(segment
-		(start 331.725 121.50625)
-		(end 327.98 121.50625)
-		(width 0.254)
-		(layer "B.Cu")

Commit message: Add silkscreen
Other:
- board text added: "80% ProMicro MCU Matrix Rev. 1.3"
Changed lines of the file:
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@@
 		)
+	)
+	(gr_rect
+		(start 147.11 169.1)
+		(end 171.95 175.34)
+		(stroke
+			(width 0.1)
+			(type solid)
+		)
+		(fill no)
+		(layer "B.SilkS")
 	)
 	(gr_line
@@
 		(layer "Edge.Cuts")
 	)
+	(gr_text "80% ProMicro MCU Matrix\nRev. 1.3"
+		(at 159.625 172.195 0)
+		(layer "B.SilkS")
+		(effects
+			(font
+				(size 1 1)
+				(thickness 0.15)
+			)
+			(justify mirror)
+		)
+	)
 	(segment

Commit message: Add ground zone
Parts:
- REF** (x4): value MountingHole_2.5mm -> MountingHole_2.2mm_M2_Pad_TopOnly; footprint MountingHole:MountingHole_2.5mm -> MountingHole:MountingHole_2.2mm_M2_Pad_TopOnly
Routing:
- added copper zone on F.Cu, net GND
Changed lines of the file:
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@@
 	(net 83 "unconnected-(U1-RST-Pad22)")
 	(net 84 "GND")
-	(footprint "MountingHole:MountingHole_2.5mm"
+	(footprint "MountingHole:MountingHole_2.2mm_M2_Pad_TopOnly"
 		(layer "F.Cu")
 		(at 311.45 115.29)
-		(descr "Mounting Hole 2.5mm, no annular, generated by kicad-footprint-generator mountinghole.py")
-		(tags "mountinghole")
+		(descr "Mounting Hole 2.2mm, M2, generated by kicad-footprint-generator mountinghole.py")
+		(tags "mountinghole M2")
 		(property "Reference" "REF**"
-			(at 0 -3.45 0)
+			(at 0 -3.15 0)
 			(layer "F.SilkS")
 			(hide yes)
@@
 			)
 		)
-		(property "Value" "MountingHole_2.5mm"
-			(at 0 3.45 0)
+		(property "Value" "MountingHole_2.2mm_M2_Pad_TopOnly"
+			(at 0 3.15 0)
 			(layer "F.Fab")
 			(hide yes)
@@
 		(fp_circle
 			(center 0 0)
-			(end 2.5 0)
+			(end 2.2 0)
 			(stroke
 				(width 0.15)
@@
 		(fp_circle
 			(center 0 0)
-			(end 2.75 0)
+			(end 2.45 0)
 			(stroke
 				(width 0.05)
@@
 			(layer "F.CrtYd")
 		)
-		(pad "" np_thru_hole circle
+		(fp_text user "${REFERENCE}"
+			(at 0 0 0)
+			(layer "F.Fab")
+			(effects
+				(font
+					(size 1 1)
+					(thickness 0.15)
+				)
+			)
+		)
+		(pad "1" thru_hole circle
 			(at 0 0)
-			(size 2.5 2.5)
-			(drill 2.5)
+			(size 2.6 2.6)
+			(drill 2.2)
 			(layers "*.Cu" "*.Mask")
+			(remove_unused_layers no)
+			(zone_connect 2)
+		)
+		(pad "1" connect circle
+			(at 0 0)
+			(size 4.4 4.4)
+			(layers "F.Cu" "F.Mask")
+			(zone_connect 2)
 		)
 		(embedded_fonts no)
 	)
-	(footprint "MountingHole:MountingHole_2.5mm"
+	(footprint "MountingHole:MountingHole_2.2mm_M2_Pad_TopOnly"
 		(layer "F.Cu")
 		(at 77.37 114.81)
-		(descr "Mounting Hole 2.5mm, no annular, generated by kicad-footprint-generator mountinghole.py")
-		(tags "mountinghole")
+		(descr "Mounting Hole 2.2mm, M2, generated by kicad-footprint-generator mountinghole.py")
+		(tags "mountinghole M2")
 		(property "Reference" "REF**"
-			(at 0 -3.45 0)
+			(at 0 -3.15 0)
 			(layer "F.SilkS")
 			(hide yes)
@@
 			)
 		)
-		(property "Value" "MountingHole_2.5mm"
-			(at 0 3.45 0)
+		(property "Value" "MountingHole_2.2mm_M2_Pad_TopOnly"
+			(at 0 3.15 0)
 			(layer "F.Fab")
 			(hide yes)
@@
 		(fp_circle
 			(center 0 0)
-			(end 2.5 0)
+			(end 2.2 0)
 			(stroke
 				(width 0.15)
@@
 		(fp_circle
 			(center 0 0)
-			(end 2.75 0)
+			(end 2.45 0)
 			(stroke
 				(width 0.05)
@@
 			(layer "F.CrtYd")
 		)
-		(pad "" np_thru_hole circle
+		(fp_text user "${REFERENCE}"
+			(at 0 0 0)
+			(layer "F.Fab")
+			(effects
+				(font
+					(size 1 1)
+					(thickness 0.15)
+				)
+			)
+		)
+		(pad "1" thru_hole circle
 			(at 0 0)
-			(size 2.5 2.5)
-			(drill 2.5)
+			(size 2.6 2.6)
+			(drill 2.2)
 			(layers "*.Cu" "*.Mask")
+			(remove_unused_layers no)
+			(zone_connect 2)
+		)
+		(pad "1" connect circle
+			(at 0 0)
+			(size 4.4 4.4)
+			(layers "F.Cu" "F.Mask")
+			(zone_connect 2)
 		)
 		(embedded_fonts no)
 	)
-	(footprint "MountingHole:MountingHole_2.5mm"
+	(footprint "MountingHole:MountingHole_2.2mm_M2_Pad_TopOnly"
 		(layer "F.Cu")
 		(at 223.04375 172.24375)
-		(descr "Mounting Hole 2.5mm, no annular, generated by kicad-footprint-generator mountinghole.py")
-		(tags "mountinghole")
+		(descr "Mounting Hole 2.2mm, M2, generated by kicad-footprint-generator mountinghole.py")
+		(tags "mountinghole M2")
 		(property "Reference" "REF**"
-			(at 0 -3.45 0)
+			(at 0 -3.15 0)
 			(layer "F.SilkS")
 			(hide yes)
@@
 			)
 		)
-		(property "Value" "MountingHole_2.5mm"
-			(at 0 3.45 0)
+		(property "Value" "MountingHole_2.2mm_M2_Pad_TopOnly"
+			(at 0 3.15 0)
 			(layer "F.Fab")
 			(hide yes)
@@
 		(fp_circle
 			(center 0 0)
-			(end 2.5 0)
+			(end 2.2 0)
 			(stroke
 				(width 0.15)
@@
 		(fp_circle
 			(center 0 0)
-			(end 2.75 0)
+			(end 2.45 0)
 			(stroke
 				(width 0.05)
@@
 			(layer "F.CrtYd")
 		)
-		(pad "" np_thru_hole circle
+		(fp_text user "${REFERENCE}"
+			(at 0 0 0)
+			(layer "F.Fab")
+			(effects
+				(font
+					(size 1 1)
+					(thickness 0.15)
+				)
+			)
+		)
+		(pad "1" thru_hole circle
 			(at 0 0)
-			(size 2.5 2.5)
-			(drill 2.5)
+			(size 2.6 2.6)
+			(drill 2.2)
 			(layers "*.Cu" "*.Mask")
+			(remove_unused_layers no)
+			(zone_connect 2)
+		)
+		(pad "1" connect circle
+			(at 0 0)
+			(size 4.4 4.4)
+			(layers "F.Cu" "F.Mask")
+			(zone_connect 2)
 		)
 		(embedded_fonts no)
 	)
-	(footprint "MountingHole:MountingHole_2.5mm"
+	(footprint "MountingHole:MountingHole_2.2mm_M2_Pad_TopOnly"
 		(layer "F.Cu")
 		(at 142.08 172.24375)
-		(descr "Mounting Hole 2.5mm, no annular, generated by kicad-footprint-generator mountinghole.py")
-		(tags "mountinghole")
+		(descr "Mounting Hole 2.2mm, M2, generated by kicad-footprint-generator mountinghole.py")
+		(tags "mountinghole M2")
 		(property "Reference" "REF**"
-			(at 0 -3.45 0)
+			(at 0 -3.15 0)
 			(layer "F.SilkS")
 			(hide yes)
@@
 			)
 		)
-		(property "Value" "MountingHole_2.5mm"
-			(at 0 3.45 0)
+		(property "Value" "MountingHole_2.2mm_M2_Pad_TopOnly"
+			(at 0 3.15 0)
 			(layer "F.Fab")
 			(hide yes)
@@
 		(fp_circle
 			(center 0 0)
-			(end 2.5 0)
+			(end 2.2 0)
 			(stroke
 				(width 0.15)
@@
 		(fp_circle
 			(center 0 0)
-			(end 2.75 0)
+			(end 2.45 0)
 			(stroke
 				(width 0.05)
@@
 			(layer "F.CrtYd")
 		)
-		(pad "" np_thru_hole circle
+		(fp_text user "${REFERENCE}"
+			(at 0 0 0)
+			(layer "F.Fab")
+			(effects
+				(font
+					(size 1 1)
+					(thickness 0.15)
+				)
+			)
+		)
+		(pad "1" thru_hole circle
 			(at 0 0)
-			(size 2.5 2.5)
-			(drill 2.5)
+			(size 2.6 2.6)
+			(drill 2.2)
 			(layers "*.Cu" "*.Mask")
+			(remove_unused_layers no)
+			(net 84 "GND")
+			(zone_connect 2)
+		)
+		(pad "1" connect circle
+			(at 0 0)
+			(size 4.4 4.4)
+			(layers "F.Cu" "F.Mask")
+			(net 84 "GND")
+			(zone_connect 2)
 		)
 		(embedded_fonts no)
@@
 	)
 	(segment
-		(start 151.60625 171.45)
-		(end 151.60625 151.79675)
-		(width 0.254)
-		(layer "F.Cu")
-		(net 70)
-	)
-	(segment
 		(start 143.16075 90.96375)
 		(end 143.35125 90.96375)
@@
 	)
 	(segment
-		(start 157.1625 177.00625)
-		(end 151.60625 171.45)
-		(width 0.254)
-		(layer "F.Cu")
-		(net 70)
-	)
-	(segment
 		(start 157.44825 120.142)
 		(end 157.44825 129.06375)
@@
 	)
 	(segment
-		(start 209.76 179.86375)
-		(end 206.9025 177.00625)
+		(start 151.60625 171.45)
+		(end 151.60625 151.79675)
 		(width 0.254)
 		(layer "F.Cu")
@@
 	)
 	(segment
-		(start 151.60625 151.79675)
-		(end 147.92325 148.11375)
+		(start 205.315 175.41875)
+		(end 155.575 175.41875)
 		(width 0.254)
 		(layer "F.Cu")
@@
 	)
 	(segment
-		(start 206.9025 177.00625)
-		(end 157.1625 177.00625)
+		(start 143.35125 90.96375)
+		(end 146.84375 94.45625)
 		(width 0.254)
 		(layer "F.Cu")
@@
 	)
 	(segment
-		(start 143.35125 90.96375)
-		(end 146.84375 94.45625)
+		(start 209.76 179.86375)
+		(end 205.315 175.41875)
+		(width 0.254)
+		(layer "F.Cu")
+		(net 70)
+	)
+	(segment
+		(start 155.575 175.41875)
+		(end 151.60625 171.45)
+		(width 0.254)
+		(layer "F.Cu")
+		(net 70)
+	)
+	(segment
+		(start 151.60625 151.79675)
+		(end 147.92325 148.11375)
 		(width 0.254)
 		(layer "F.Cu")
@@
 		(net 82)
 	)
+	(zone
+		(net 84)
+		(net_name "GND")
+		(layer "F.Cu")
+		(hatch edge 0.5)
+		(connect_pads
+			(clearance 0.5)
+		)
+		(min_thickness 0.25)
+		(filled_areas_thickness no)
+		(fill yes
+			(thermal_gap 0.5)
+			(thermal_bridge_width 0.5)
+		)
+		(polygon
+			(pts
+				(xy 137.31875 167.48125) (xy 146.05 167.48125) (xy 154.768651 176.199901) (xy 205.58125 176.2125)
+				(xy 208.75625 179.3875) (xy 208.75625 180.18125) (xy 203.2 180.18125) (xy 203.2 178.59375) (xy 137.31875 178.59375)
+			)
+		)
+	)
 	(group ""

Commit message: Set all pads to top only
Parts:
- REF** (x4): value MountingHole_2.2mm_M2_Pad_TopOnly -> MountingHole_2.5mm_Pad_TopOnly; footprint MountingHole:MountingHole_2.2mm_M2_Pad_TopOnly -> MountingHole:MountingHole_2.5mm_Pad_TopOnly
Connections:
- REF** pad 1: GND -> (no net)
Routing:
- removed copper zone on F.Cu, net GND
Changed lines of the file:
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@@
 	(net 83 "unconnected-(U1-RST-Pad22)")
 	(net 84 "GND")
-	(footprint "MountingHole:MountingHole_2.2mm_M2_Pad_TopOnly"
+	(footprint "MountingHole:MountingHole_2.5mm_Pad_TopOnly"
 		(layer "F.Cu")
 		(at 311.45 115.29)
-		(descr "Mounting Hole 2.2mm, M2, generated by kicad-footprint-generator mountinghole.py")
-		(tags "mountinghole M2")
+		(descr "Mounting Hole 2.5mm, generated by kicad-footprint-generator mountinghole.py")
+		(tags "mountinghole")
 		(property "Reference" "REF**"
-			(at 0 -3.15 0)
+			(at 0 -3.45 0)
 			(layer "F.SilkS")
 			(hide yes)
@@
 			)
 		)
-		(property "Value" "MountingHole_2.2mm_M2_Pad_TopOnly"
-			(at 0 3.15 0)
+		(property "Value" "MountingHole_2.5mm_Pad_TopOnly"
+			(at 0 3.45 0)
 			(layer "F.Fab")
 			(hide yes)
@@
 		(fp_circle
 			(center 0 0)
-			(end 2.2 0)
+			(end 2.5 0)
 			(stroke
 				(width 0.15)
@@
 		(fp_circle
 			(center 0 0)
-			(end 2.45 0)
+			(end 2.75 0)
 			(stroke
 				(width 0.05)
@@
 		(pad "1" thru_hole circle
 			(at 0 0)
-			(size 2.6 2.6)
-			(drill 2.2)
+			(size 2.9 2.9)
+			(drill 2.5)
 			(layers "*.Cu" "*.Mask")
 			(remove_unused_layers no)
@@
 		(pad "1" connect circle
 			(at 0 0)
-			(size 4.4 4.4)
+			(size 5 5)
 			(layers "F.Cu" "F.Mask")
 			(zone_connect 2)
@@
 		(embedded_fonts no)
 	)
-	(footprint "MountingHole:MountingHole_2.2mm_M2_Pad_TopOnly"
+	(footprint "MountingHole:MountingHole_2.5mm_Pad_TopOnly"
 		(layer "F.Cu")
 		(at 77.37 114.81)
-		(descr "Mounting Hole 2.2mm, M2, generated by kicad-footprint-generator mountinghole.py")
-		(tags "mountinghole M2")
+		(descr "Mounting Hole 2.5mm, generated by kicad-footprint-generator mountinghole.py")
+		(tags "mountinghole")
 		(property "Reference" "REF**"
-			(at 0 -3.15 0)
+			(at 0 -3.45 0)
 			(layer "F.SilkS")
 			(hide yes)
@@
 			)
 		)
-		(property "Value" "MountingHole_2.2mm_M2_Pad_TopOnly"
-			(at 0 3.15 0)
+		(property "Value" "MountingHole_2.5mm_Pad_TopOnly"
+			(at 0 3.45 0)
 			(layer "F.Fab")
 			(hide yes)
@@
 		(fp_circle
 			(center 0 0)
-			(end 2.2 0)
+			(end 2.5 0)
 			(stroke
 				(width 0.15)
@@
 		(fp_circle
 			(center 0 0)
-			(end 2.45 0)
+			(end 2.75 0)
 			(stroke
 				(width 0.05)
@@
 		(pad "1" thru_hole circle
 			(at 0 0)
-			(size 2.6 2.6)
-			(drill 2.2)
+			(size 2.9 2.9)
+			(drill 2.5)
 			(layers "*.Cu" "*.Mask")
 			(remove_unused_layers no)
@@
 		(pad "1" connect circle
 			(at 0 0)
-			(size 4.4 4.4)
+			(size 5 5)
 			(layers "F.Cu" "F.Mask")
 			(zone_connect 2)
@@
 		(embedded_fonts no)
 	)
-	(footprint "MountingHole:MountingHole_2.2mm_M2_Pad_TopOnly"
+	(footprint "MountingHole:MountingHole_2.5mm_Pad_TopOnly"
 		(layer "F.Cu")
 		(at 223.04375 172.24375)
-		(descr "Mounting Hole 2.2mm, M2, generated by kicad-footprint-generator mountinghole.py")
-		(tags "mountinghole M2")
+		(descr "Mounting Hole 2.5mm, generated by kicad-footprint-generator mountinghole.py")
+		(tags "mountinghole")
 		(property "Reference" "REF**"
-			(at 0 -3.15 0)
+			(at 0 -3.45 0)
 			(layer "F.SilkS")
 			(hide yes)
@@
 			)
 		)
-		(property "Value" "MountingHole_2.2mm_M2_Pad_TopOnly"
-			(at 0 3.15 0)
+		(property "Value" "MountingHole_2.5mm_Pad_TopOnly"
+			(at 0 3.45 0)
 			(layer "F.Fab")
 			(hide yes)
@@
 		(fp_circle
 			(center 0 0)
-			(end 2.2 0)
+			(end 2.5 0)
 			(stroke
 				(width 0.15)
@@
 		(fp_circle
 			(center 0 0)
-			(end 2.45 0)
+			(end 2.75 0)
 			(stroke
 				(width 0.05)
@@
 		(pad "1" thru_hole circle
 			(at 0 0)
-			(size 2.6 2.6)
-			(drill 2.2)
+			(size 2.9 2.9)
+			(drill 2.5)
 			(layers "*.Cu" "*.Mask")
 			(remove_unused_layers no)
@@
 		(pad "1" connect circle
 			(at 0 0)
-			(size 4.4 4.4)
+			(size 5 5)
 			(layers "F.Cu" "F.Mask")
 			(zone_connect 2)
@@
 		(embedded_fonts no)
 	)
-	(footprint "MountingHole:MountingHole_2.2mm_M2_Pad_TopOnly"
+	(footprint "MountingHole:MountingHole_2.5mm_Pad_TopOnly"
 		(layer "F.Cu")
 		(at 142.08 172.24375)
-		(descr "Mounting Hole 2.2mm, M2, generated by kicad-footprint-generator mountinghole.py")
-		(tags "mountinghole M2")
+		(descr "Mounting Hole 2.5mm, generated by kicad-footprint-generator mountinghole.py")
+		(tags "mountinghole")
 		(property "Reference" "REF**"
-			(at 0 -3.15 0)
+			(at 0 -3.45 0)
 			(layer "F.SilkS")
 			(hide yes)
@@
 			)
 		)
-		(property "Value" "MountingHole_2.2mm_M2_Pad_TopOnly"
-			(at 0 3.15 0)
+		(property "Value" "MountingHole_2.5mm_Pad_TopOnly"
+			(at 0 3.45 0)
 			(layer "F.Fab")
 			(hide yes)
@@
 		(fp_circle
 			(center 0 0)
-			(end 2.2 0)
+			(end 2.5 0)
 			(stroke
 				(width 0.15)
@@
 		(fp_circle
 			(center 0 0)
-			(end 2.45 0)
+			(end 2.75 0)
 			(stroke
 				(width 0.05)
@@
 		(pad "1" thru_hole circle
 			(at 0 0)
-			(size 2.6 2.6)
-			(drill 2.2)
+			(size 2.9 2.9)
+			(drill 2.5)
 			(layers "*.Cu" "*.Mask")
 			(remove_unused_layers no)
-			(net 84 "GND")
 			(zone_connect 2)
 		)
 		(pad "1" connect circle
 			(at 0 0)
-			(size 4.4 4.4)
+			(size 5 5)
 			(layers "F.Cu" "F.Mask")
-			(net 84 "GND")
 			(zone_connect 2)
 		)
@@
 	)
 	(segment
+		(start 151.60625 171.45)
+		(end 151.60625 151.79675)
+		(width 0.254)
+		(layer "F.Cu")
+		(net 70)
+	)
+	(segment
 		(start 143.16075 90.96375)
 		(end 143.35125 90.96375)
@@
 	)
 	(segment
+		(start 157.1625 177.00625)
+		(end 151.60625 171.45)
+		(width 0.254)
+		(layer "F.Cu")
+		(net 70)
+	)
+	(segment
 		(start 157.44825 120.142)
 		(end 157.44825 129.06375)
@@
 	)
 	(segment
-		(start 151.60625 171.45)
-		(end 151.60625 151.79675)
-		(width 0.254)
-		(layer "F.Cu")
-		(net 70)
-	)
-	(segment
-		(start 205.315 175.41875)
-		(end 155.575 175.41875)
-		(width 0.254)
-		(layer "F.Cu")
-		(net 70)
-	)
-	(segment
-		(start 143.35125 90.96375)
-		(end 146.84375 94.45625)
+		(start 209.76 179.86375)
+		(end 206.9025 177.00625)
 		(width 0.254)
 		(layer "F.Cu")
@@
 	)
 	(segment
-		(start 209.76 179.86375)
-		(end 205.315 175.41875)
+		(start 151.60625 151.79675)
+		(end 147.92325 148.11375)
 		(width 0.254)
 		(layer "F.Cu")
@@
 	)
 	(segment
-		(start 155.575 175.41875)
-		(end 151.60625 171.45)
+		(start 206.9025 177.00625)
+		(end 157.1625 177.00625)
 		(width 0.254)
 		(layer "F.Cu")
@@
 	)
 	(segment
-		(start 151.60625 151.79675)
-		(end 147.92325 148.11375)
+		(start 143.35125 90.96375)
+		(end 146.84375 94.45625)
 		(width 0.254)
 		(layer "F.Cu")
@@
 		(net 82)
 	)
-	(zone
-		(net 84)
-		(net_name "GND")
-		(layer "F.Cu")
-		(hatch edge 0.5)
-		(connect_pads
-			(clearance 0.5)
-		)
-		(min_thickness 0.25)
-		(filled_areas_thickness no)
-		(fill yes
-			(thermal_gap 0.5)
-			(thermal_bridge_width 0.5)
-		)
-		(polygon
-			(pts
-				(xy 137.31875 167.48125) (xy 146.05 167.48125) (xy 154.768651 176.199901) (xy 205.58125 176.2125)
-				(xy 208.75625 179.3875) (xy 208.75625 180.18125) (xy 203.2 180.18125) (xy 203.2 178.59375) (xy 137.31875 178.59375)
-			)
-		)
-	)
 	(group ""

Commit message: Start moving vias to be adjacent to pads
Routing:
- net Col12: track 201.2 -> 206.6 mm
- net Col3: track 182.3 -> 183.6 mm
- net Col2: track 182.7 -> 184.0 mm
- net Col8: track 161.7 -> 163.0 mm
- net Col7: track 139.5 -> 140.7 mm
- net Col0: track 247.8 -> 249.1 mm
- net Col10: track 236.8 -> 238.0 mm
- net Col9: track 199.0 -> 200.2 mm
- net Col5: track 124.9 -> 126.2 mm
- net Col1: track 231.5 -> 232.7 mm
- net Col6: track 105.9 -> 107.0 mm
- net Col4: track 154.7 -> 153.8 mm
Other:
- board text added: "80% ProMicro MCU Matrix Rev. 1.4"
- board text removed: "80% ProMicro MCU Matrix Rev. 1.3"

Commit message: More via tweaks
Routing:
- net Col3: track 183.6 -> 174.3 mm
- net Col2: track 184.0 -> 191.8 mm
- net Col4: track 153.8 -> 147.7 mm
- net Col0: track 249.1 -> 254.4 mm
- net Col8: track 163.0 -> 167.1 mm
- net Col9: track 200.2 -> 204.4 mm
- net Col7: track 140.7 -> 144.9 mm
- net Col10: track 238.0 -> 241.7 mm
- net Col5: track 126.2 -> 128.3 mm
- net Col1: track 232.7 -> 234.6 mm
Other:
- board text added: "80% ProMicro MCU Matrix Rev. 1.3"
- board text removed: "80% ProMicro MCU Matrix Rev. 1.4"

Commit message: One row left!
Routing:
- net Col3: track 174.3 -> 188.1 mm
- net Col4: track 147.7 -> 160.3 mm
- net Col12: track 206.6 -> 219.2 mm
- net Col11: track 229.8 -> 236.3 mm
- net Col10: track 241.7 -> 247.2 mm
- net Col8: track 167.1 -> 172.3 mm
- net Col7: track 144.9 -> 149.3 mm
- net Col6: track 107.0 -> 111.4 mm
- net Col5: track 128.3 -> 132.6 mm
- net Col0: track 254.4 -> 258.6 mm
- net Col1: track 234.6 -> 238.7 mm
- net Col9: track 204.4 -> 206.0 mm
